Commit message: added ros controller for simuated ur5

File: simulation/ur_simulation/ur_gazebo/urdf/ur.urdf.xacro (robot description, xacro)
@@ -38,6 +38,6 @@
    <xacro:arg name="fake_sensor_commands" default="false" />
    <xacro:arg name="sim_gazebo" default="false" />
-   <xacro:arg name="sim_ignition" default="false" />
-   <xacro:arg name="simulation_controllers" default="" />
+   <xacro:arg name="sim_ignition" default="true" />
+   <xacro:arg name="simulation_controllers" default="$(find ur_gazebo)/config/controller_configuration.yaml" />
    <!-- initial position for simulations (Fake Hardware, Gazebo, Ignition) -->
    <xacro:arg name="initial_positions_file" default="$(find ur_description)/config/initial_positions.yaml"/>
@@ -93,4 +93,5 @@
   <xacro:if value="$(arg sim_ignition)">
     <!-- Gazebo plugins -->
+    <!-- This seems to be working only with edifice not fortress.
     <gazebo reference="world">
     </gazebo>
@@ -101,4 +102,28 @@
       </plugin>
     </gazebo>
+    -->
+<!-- This block does seem necessary for the ignition simulation + ros2_conrol to work
+  <ros2_control name="IgnitionSystem" type="system">
+    <hardware>
+      <plugin>ign_ros2_control/IgnitionSystem</plugin>
+    </hardware>
+    <joint name="shoulder_pan_joint">
+      <command_interface name="position">
+        <param name="min">-3.1415926</param>
+        <param name="max">3.1415926</param>
+      </command_interface>
+      <state_interface name="position"/>
+      <state_interface name="velocity"/>
+      <state_interface name="effort"/>
+    </joint>
+  </ros2_control>
+-->
+  <gazebo>
+    <plugin filename="libign_ros2_control-system.so" name="ign_ros2_control::IgnitionROS2ControlPlugin">
+      <robot_param>robot_description</robot_param>
+      <robot_param_node>robot_state_publisher</robot_param_node>
+      <parameters>$(arg simulation_controllers)</parameters>
+    </plugin>
+  </gazebo>
   </xacro:if>
   <!-- Joint state publisher-->

Commit message: added gripper to end effctor, improved camera resolution

File: simulation/ur_simulation/ur_gazebo/urdf/ur.urdf.xacro (robot description, xacro)
@@ -81,5 +81,10 @@
      <origin xyz="0 0 0" rpy="0 0 0" />          <!-- position robot in the world -->
    </xacro:ur_robot>
-   <xacro:if value="$(arg sim_gazebo)">
+  <!-- include gripper xacro file -->
+  <xacro:include filename="$(find ur_gazebo)/urdf/robotiq_gripper.xacro" />
+  <!-- gripper -->
+  <xacro:robotiq_gripper mount="tool0">  <!-- attach to tool0 -->
+  </xacro:robotiq_gripper>
+  <xacro:if value="$(arg sim_gazebo)">
     <!-- Gazebo plugins -->
     <gazebo reference="world">
@@ -92,31 +97,4 @@
   </xacro:if>
   <xacro:if value="$(arg sim_ignition)">
-    <!-- Gazebo plugins -->
-    <!-- This seems to be working only with edifice not fortress.
-    <gazebo reference="world">
-    </gazebo>
-    <gazebo>
-      <plugin filename="libign_ros2_control-system.so" name="ign_ros2_control::IgnitionROS2ControlPlugin">
-        <parameters>$(arg simulation_controllers)</parameters>
-        <controller_manager_node_name>$(arg prefix)controller_manager</controller_manager_node_name>
-      </plugin>
-    </gazebo>
-    -->
-<!-- This block does seem necessary for the ignition simulation + ros2_conrol to work
-  <ros2_control name="IgnitionSystem" type="system">
-    <hardware>
-      <plugin>ign_ros2_control/IgnitionSystem</plugin>
-    </hardware>
-    <joint name="shoulder_pan_joint">
-      <command_interface name="position">
-        <param name="min">-3.1415926</param>
-        <param name="max">3.1415926</param>
-      </command_interface>
-      <state_interface name="position"/>
-      <state_interface name="velocity"/>
-      <state_interface name="effort"/>
-    </joint>
-  </ros2_control>
--->
   <gazebo>
     <plugin filename="libign_ros2_control-system.so" name="ign_ros2_control::IgnitionROS2ControlPlugin">

Commit message: Added camera3 onto wrist_3_link

File: simulation/ur_simulation/ur_gazebo/urdf/ur.urdf.xacro (robot description, xacro)
@@ -86,4 +86,10 @@
   <xacro:robotiq_gripper mount="tool0">  <!-- attach to tool0 -->
   </xacro:robotiq_gripper>
+  <!-- include ur_sim_camera xacro file-->
+  <xacro:include filename="$(find ur_gazebo)/urdf/ur_sim_camera.xacro" />
+  <!-- camera mount on wrist3 -->
+  <xacro:ur_sim_camera name="camera3" parent="wrist_3_link">
+    <origin xyz="0.0 -0.05 0.0" rpy="0.0 0.0 0.0" />
+  </xacro:ur_sim_camera>
   <xacro:if value="$(arg sim_gazebo)">
     <!-- Gazebo plugins -->

File: simulation/ur_simulation/ur_gazebo/urdf/ur_sim_camera.xacro (robot description, xacro)
@@ -3,9 +3,13 @@
         <link name="camera_body">
             <xacro:insert_block name="origin"/>
+            <inertial>
+              <origin xyz="0 0 0" rpy="0 0 0"/>
+              <mass value="0.01"/>
+              <inertia ixx="0.1"  ixy="0"  ixz="0" iyy="0.1" iyz="0" izz="0.1" />
+            </inertial>
             <visual>
-                <origin xyz="0 0 0" rpy="1.57 0 1.57"/>
+                <origin xyz="0 0 0" rpy="0 0 0"/>
                 <geometry>
-                    <!--Orient the model to look forward-->
-                    <mesh filename="file://$(find ur_gazebo)/meshes/Camera.obj" scale="0.001 0.001 0.001" />
+                    <box size="0.05 0.02 0.02"/>
                 </geometry>
                 <material name="Grey">
@@ -15,5 +19,5 @@
             <collision>
                 <geometry>
-                    <mesh filename="file://$(find ur_gazebo)/meshes/Camera.obj" scale="0.001 0.001 0.001" />
+                    <box size="0.05 0.02 0.02"/>
                 </geometry>
             </collision>
@@ -26,24 +30,21 @@
         <gazebo reference="camera_body">
             <sensor name="${name}" type="camera">
-                <ignition_frame_id>base_link</ignition_frame_id>
-                <update_rate>40.0</update_rate>
-                <always_on>1</always_on>
-                <topic> camera </topic>
-                <camera name="camera">
+                <pose>0 0 0 -1.5707 -1.5707 3.14159</pose>
+                <camera>
                     <horizontal_fov>1.047</horizontal_fov>
                     <image>
-                        <width>640</width>
-                        <height>480</height>
+                        <width>960</width>
+                        <height>720</height>
                         <format>R8G8B8</format>
                     </image>
                     <clip>
-                        <near>0.1</near>
-                        <far>100</far>
+                        <near>0.02</near>
+                        <far>300</far>
                     </clip>
                 </camera>
+                <always_on>1</always_on>
+                <update_rate>30</update_rate>
                 <visualize>true</visualize>
-                	<plugin filename="ignition-gazebo-sensors-system"
-                        name="ignition::gazebo::systems::Sensors">
-                    </plugin>
+                <topic>image3</topic>
             </sensor>
         </gazebo>

Commit message: Added depth camera detups

File: simulation/ur_simulation/ur_gazebo/urdf/ur.urdf.xacro (robot description, xacro)
@@ -1,4 +1,4 @@
 <?xml version="1.0"?>
-<robot xmlns:xacro="http://wiki.ros.org/xacro" name="$(arg name)">
+<robot xmlns:xacro="http://wiki.ros.org/xacro" name="ur">
    <!-- robot name parameter -->
    <xacro:arg name="name" default="ur"/>
@@ -7,5 +7,5 @@
    <!-- possible 'ur_type' values: ur3, ur3e, ur5, ur5e, ur10, ur10e, ur16e -->
    <!-- the default value should raise an error in case this was called without defining the type -->
-   <xacro:arg name="ur_type" default="ur5x"/>
+   <xacro:arg name="ur_type" default="ur5"/>
    <!-- parameters -->
    <xacro:arg name="prefix" default="" />
@@ -92,4 +92,7 @@
     <origin xyz="0.0 -0.05 0.0" rpy="0.0 0.0 0.0" />
   </xacro:ur_sim_camera>
+  <xacro:ur_depth_camera name="camera3_depth" parent="wrist_3_link">
+    <origin xyz="0.0 -0.05 0.0" rpy="0.0 0.0 0.0" />
+  </xacro:ur_depth_camera>
   <xacro:if value="$(arg sim_gazebo)">
     <!-- Gazebo plugins -->

File: simulation/ur_simulation/ur_gazebo/urdf/ur_sim_camera.xacro (robot description, xacro)
@@ -46,5 +46,69 @@
                 <update_rate>30</update_rate>
                 <visualize>true</visualize>
-                <topic>image3</topic>
+                <topic>/rgbd_camera/image</topic>
+            </sensor>
+        </gazebo>
+    </xacro:macro>
+    <xacro:macro name="ur_depth_camera" params="name parent *origin">
+        <link name="camera_depth_body">
+            <xacro:insert_block name="origin"/>
+            <inertial>
+              <origin xyz="0 0 0" rpy="0 0 0"/>
+              <mass value="0.01"/>
+              <inertia ixx="0.1"  ixy="0"  ixz="0" iyy="0.1" iyz="0" izz="0.1" />
+            </inertial>
+            <visual>
+                <origin xyz="0 0 0" rpy="0 0 0"/>
+                <geometry>
+                    <box size="0.05 0.02 0.02"/>
+                </geometry>
+                <material name="Grey">
+                    <color rgba="0.5 0.5 0.5 1.0"/>
+                </material>
+            </visual>
+            <collision>
+                <geometry>
+                    <box size="0.05 0.02 0.02"/>
+                </geometry>
+            </collision>
+        </link>
+        <joint name="camera_depth_link" type="fixed">
+            <parent link="${parent}"/>
+            <child link="camera_depth_body"/>
+            <xacro:insert_block name="origin"/>
+        </joint>
+        <link name="RGBD_optical_link">
+            <inertial>
+                <origin xyz="0 0 0" rpy="0 0 0"/>
+                <mass value="0.001"/>
+                <inertia ixx="0.0001"  ixy="0"  ixz="0" iyy="0.0001" iyz="0" izz="0.0001" />
+            </inertial>
+        </link>
+        <!-- New fixed joint connecting the camera_depth_body link to the RGBD_optical_link -->
+        <joint name="RGBD_optical_joint" type="fixed">
+            <parent link="camera_depth_body"/>
+            <child link="RGBD_optical_link"/>
+            <origin xyz="0 0 0" rpy="-1.5707 -1.5707 3.14159"/>
+        </joint>
+        <gazebo reference="camera_depth_body">
+            <sensor name="${name}" type="depth">
+                <pose>0 0 0 -1.5707 -1.5707 3.14159</pose>
+                <camera>
+                    <horizontal_fov>1.047</horizontal_fov>
+                    <image>
+                        <width>960</width>
+                        <height>720</height>
+                        <format>R_FLOAT32</format>
+                        <!-- <format>R8G8B8</format> -->
+                    </image>
+                    <clip>
+                        <near>0.02</near>
+                        <far>300</far>
+                    </clip>
+                </camera>
+                <always_on>1</always_on>
+                <update_rate>30</update_rate>
+                <visualize>true</visualize>
+                <topic>/rgbd_camera/depth_image</topic>
             </sensor>
         </gazebo>
