Commit message: Added stereo_vision_service; fixed depth camera format issue; renamed entry points

File: simulation/ur_simulation/ur_gazebo/urdf/ur_sim_camera.xacro (robot description, xacro)
@@ -46,5 +46,4 @@
                 <update_rate>30</update_rate>
                 <visualize>true</visualize>
-                <topic>/rgbd_camera/image</topic>
             </sensor>
         </gazebo>
@@ -89,8 +88,8 @@
             <parent link="camera_depth_body"/>
             <child link="RGBD_optical_link"/>
-            <origin xyz="0 0 0" rpy="-1.5707 -1.5707 3.14159"/>
+            <origin xyz="0 0 0" rpy="0 0 0"/>
         </joint>
         <gazebo reference="camera_depth_body">
-            <sensor name="${name}" type="depth">
+            <sensor name="${name}" type="depth_camera">
                 <pose>0 0 0 -1.5707 -1.5707 3.14159</pose>
                 <camera>
@@ -99,10 +98,8 @@
                         <width>960</width>
                         <height>720</height>
-                        <format>R_FLOAT32</format>
-                        <!-- <format>R8G8B8</format> -->
                     </image>
                     <clip>
                         <near>0.02</near>
-                        <far>2</far>
+                        <far>300</far>
                     </clip>
                 </camera>
@@ -110,5 +107,4 @@
                 <update_rate>30</update_rate>
                 <visualize>true</visualize>
-                <topic>/rgbd_camera/depth_image</topic>
             </sensor>
         </gazebo>
