Commit message: Configured MoveIt to work with gazebo simulation

File: simulation/ur_simulation/ur_gazebo/urdf/robotiq_gripper.xacro (robot description, xacro)
@@ -254,4 +254,37 @@
             <child
             link="right_inner_finger" />
+            <axis
+            xyz="0 1 0" />
+            <limit
+            lower="0"
+            upper="0.8757"
+            velocity="2.0"
+            effort="1000" />
+        </joint>
+        <!-- Add a fixed gripper_pick frame between the left finger and right finger-->
+        <link name = "gripper_pick">
+            <inertial>
+            <origin
+                xyz="0 0 0"
+                rpy="0 0 0" />
+            <mass
+                value="0.01" />
+            <inertia
+                ixx="0.001"
+                ixy="0.001"
+                ixz="0.00"
+                iyy="0.00"
+                iyz="0.00"
+                izz="0.00" />
+            </inertial>
+        </link>
+        <joint name="gripper_pick_joint" type="fixed">
+            <origin
+            xyz="0 0 0.13"
+            rpy="0 0 0" />
+            <parent
+            link="tool0" />
+            <child
+            link="gripper_pick" />
             <axis
             xyz="0 1 0" />

File: simulation/ur_simulation/ur_gazebo/urdf/ur.urdf.xacro (robot description, xacro)
@@ -35,9 +35,9 @@
    <xacro:arg name="tool_tcp_port" default="54321" />
      <!-- Simulation parameters -->
-   <xacro:arg name="use_fake_hardware" default="false" />
+   <xacro:arg name="use_fake_hardware" default="true" />
    <xacro:arg name="fake_sensor_commands" default="false" />
    <xacro:arg name="sim_gazebo" default="false" />
    <xacro:arg name="sim_ignition" default="true" />
-   <xacro:arg name="simulation_controllers" default="$(find ur_gazebo)/config/controller_configuration.yaml" />
+   <xacro:arg name="simulation_controllers" default="$(find ur5_gripper_moveit_config)/config/ros_controllers.yaml" />
    <!-- initial position for simulations (Fake Hardware, Gazebo, Ignition) -->
    <xacro:arg name="initial_positions_file" default="$(find ur_description)/config/initial_positions.yaml"/>

Commit message: gpt_rtt_demo

File: simulation/ur_simulation/ur_gazebo/urdf/robotiq_gripper.xacro (robot description, xacro)
@@ -254,37 +254,4 @@
             <child
             link="right_inner_finger" />
-            <axis
-            xyz="0 1 0" />
-            <limit
-            lower="0"
-            upper="0.8757"
-            velocity="2.0"
-            effort="1000" />
-        </joint>
-        <!-- Add a fixed gripper_pick frame between the left finger and right finger-->
-        <link name = "gripper_pick">
-            <inertial>
-            <origin
-                xyz="0 0 0"
-                rpy="0 0 0" />
-            <mass
-                value="0.01" />
-            <inertia
-                ixx="0.001"
-                ixy="0.001"
-                ixz="0.00"
-                iyy="0.00"
-                iyz="0.00"
-                izz="0.00" />
-            </inertial>
-        </link>
-        <joint name="gripper_pick_joint" type="fixed">
-            <origin
-            xyz="0 0 0.13"
-            rpy="0 0 0" />
-            <parent
-            link="tool0" />
-            <child
-            link="gripper_pick" />
             <axis
             xyz="0 1 0" />

File: simulation/ur_simulation/ur_gazebo/urdf/ur.urdf.xacro (robot description, xacro)
@@ -35,9 +35,9 @@
    <xacro:arg name="tool_tcp_port" default="54321" />
      <!-- Simulation parameters -->
-   <xacro:arg name="use_fake_hardware" default="true" />
+   <xacro:arg name="use_fake_hardware" default="false" />
    <xacro:arg name="fake_sensor_commands" default="false" />
    <xacro:arg name="sim_gazebo" default="false" />
    <xacro:arg name="sim_ignition" default="true" />
-   <xacro:arg name="simulation_controllers" default="$(find ur5_gripper_moveit_config)/config/ros_controllers.yaml" />
+   <xacro:arg name="simulation_controllers" default="$(find ur_gazebo)/config/controller_configuration.yaml" />
    <!-- initial position for simulations (Fake Hardware, Gazebo, Ignition) -->
    <xacro:arg name="initial_positions_file" default="$(find ur_description)/config/initial_positions.yaml"/>
